Commit message: updated syncing between diffcloth simulation and pybullet rendering

File: tie/tie.urdf (robot description, URDF)
Before this commit: robot tie, 1 links, 0 joints
Links:
- link Base: geometry collision mesh filename=tie.obj scale=0.15 0.15 0.15; visual mesh filename=tie.obj scale=0.15 0.15 0.15

Commit message: add perturb check, parallel render, pcd shuffle

File: tie/tie.urdf (robot description, URDF)
Before this commit: robot tie, 1 links, 0 joints
Links:
- link Base: geometry collision mesh filename=./tie/tie.obj scale=0.25 0.25 0.25; visual mesh filename=./tie/tie.obj scale=0.25 0.25 0.25
